Commit message: feat: add tb4_autonomy package with arrow-based navigation pipeline
- ArrowDetector with direction-guided tip-finding for continuous angle
- StateMachine FSM: SEARCH → ALIGN → APPROACH → READ → TURN → COOLDOWN
- MotionController with P-controller yaw turning
- VisionControllerNode wiring perception to control
- Updated root README with build/launch commands
- Added tb4_autonomy README with architecture docs

File: src/resource/tb4_raw.urdf (robot description, URDF)
Before this commit: robot turtlebot4, 48 links, 47 joints
Joints:
- joint oakd_joint: origin xyz=0.0584 0.0 0.09676 -> xyz=0.0584 0.0 0.09676 rpy=0 0.25 0

Commit message: Stabilize

File: src/resource/tb4_raw.urdf (robot description, URDF)
Before this commit: robot turtlebot4, 48 links, 47 joints
Joints:
- joint oakd_joint: origin xyz=0.0584 0.0 0.09676 rpy=0 0.25 0 -> xyz=0.0584 0.0 0.09676 rpy=0 0.1 0

File: src/resource/tb4_webots.xacro (robot description, xacro)
@@ -30,26 +30,13 @@
         <gyroName>p3d gyro</gyroName>
       </plugin>
-      <plugin type="webots_ros2_control::Ros2Control" />
+      <plugin type="tb4_sim.cmd_vel_driver.CmdVelDriver">
+        <cmdVelTopic>/cmd_vel</cmdVelTopic>
+        <odomTopic>/odom</odomTopic>
+        <leftMotor>left_wheel_joint</leftMotor>
+        <rightMotor>right_wheel_joint</rightMotor>
+        <wheelSeparation>0.25</wheelSeparation>
+        <wheelRadius>0.036</wheelRadius>
+        <maxWheelSpeed>20.0</maxWheelSpeed>
+      </plugin>
     </webots>
-    <ros2_control name="WebotsControl" type="system">
-      <hardware>
-        <plugin>webots_ros2_control::Ros2ControlSystem</plugin>
-      </hardware>
-      <joint name="right_wheel_joint">
-        <command_interface name="velocity">
-            <param name="min">-20</param>
-            <param name="max">20</param>
-        </command_interface>
-        <state_interface name="position" />
-        <state_interface name="velocity" />
-      </joint>
-      <joint name="left_wheel_joint">
-        <command_interface name="velocity">
-            <param name="min">-20</param>
-            <param name="max">20</param>
-        </command_interface>
-        <state_interface name="position" />
-        <state_interface name="velocity" />
-      </joint>
-    </ros2_control>
 </robot>
